File: Q2.kicad_pcb (KiCad board)
At the start: 2 copper layers, 86 x 55 mm, 158 parts, among them U1 LM317, U10 SP-2U1+, U11 SMA, U12 LT1009, U13 TL974, U14 PMA4-33GLN+, U2 Teensy3.2, U3 SMA, U4 ROS-2536C-119+, U5 PMA4-33GLN+, U6 PGA-103+, U7 TCBT-14+, U8 SIM-43LH+, U9 GAT-7+

Commit message: Update
Parts:
- removed the REF** at (114.3, 63.5)
- removed the REF** at (38.1, 78.7)
- removed the REF** at (38.1, 73.7)
- added REF**: via-15mil, Q2Footprint:via-15mil, F.Cu at (99.1, 53.3)
- added REF**: via-15mil, Q2Footprint:via-15mil, F.Cu at (104.1, 53.3)
- added REF**: via-15mil, Q2Footprint:via-15mil, F.Cu at (109.2, 53.3)
- added REF**: via-15mil, Q2Footprint:via-15mil, F.Cu at (114.3, 53.3)
- moved U2 35.5 mm to (36.5, 76.1), turned to 270 degrees
- moved C13 5.11 mm to (113.6, 59.8)
- moved U7 0.12 mm to (101.3, 77.2)
Routing:
- net Net-(U2-Pad18): track 7.71 -> 38.5 mm
- net Net-(C13-Pad2): track 10.8 -> 5.67 mm
- net Net-(C13-Pad1): track 50.8 -> 51.4 mm

Commit message: Update
Parts:
- removed the REF** at (63.5, 33.0)
- added TP10: TEST, Q2Footprint:PINTST, F.Cu at (102.6, 81.6)
- added TP11: TEST, Q2Footprint:PINTST, F.Cu at (117.0, 71.3)
- added TP12: TEST, Q2Footprint:PINTST, F.Cu at (115.9, 64.2)
- added TP13: TEST, Q2Footprint:PINTST, F.Cu at (107.7, 76.0)
- added TP14: TEST, Q2Footprint:PINTST, F.Cu at (64.8, 32.5)
- added TP6: TEST, Q2Footprint:PINTST, F.Cu at (60.9, 57.1)
- added TP7: TEST, Q2Footprint:PINTST, F.Cu at (90.3, 81.7)
- added TP8: TEST, Q2Footprint:PINTST, F.Cu at (116.1, 58.0)
- added TP9: TEST, Q2Footprint:PINTST, F.Cu at (106.6, 68.9)
- TP1, TP2, TP3, TP4, TP5: footprint Q2Footprint:Test_Point_Keystone_5000-5004_Miniature -> Q2Footprint:PINTST
- moved TP2 1.12 mm to (37.9, 54.5)
- moved TP5 0.43 mm to (97.0, 35.8)
- moved TP1 0.27 mm to (38.0, 65.7)
- moved TP4 0.18 mm to (89.2, 42.6)
- moved TP3 0.12 mm to (37.9, 59.3)
Connections:
- U7 pad : GND -> (no net)
Routing:
- net Net-(C12-Pad1): track 3.94 -> 8.93 mm
- net Net-(R7-Pad1): track 8.41 -> 13.0 mm
- net Net-(C14-Pad2): track 13.8 -> 16.8 mm
- net Net-(TP10-Pad1): track 2.98 -> 5.83 mm
- net Net-(C7-Pad2): track 3.66 -> 6.50 mm
- net Net-(C24-Pad1): track 5.81 -> 8.53 mm
- net Net-(C13-Pad2): track 5.67 -> 8.05 mm
- net Net-(TP11-Pad1): track 5.11 -> 7.32 mm
- net Net-(TP13-Pad1): track 4.36 -> 6.26 mm

Commit message: Update
Parts:
- moved TP7 0.65 mm to (89.7, 81.6)
- moved C7 0.64 mm to (90.9, 78.9)
- moved TP13 0.44 mm to (107.7, 75.5)
- moved U6 0.41 mm to (96.2, 76.9)
- moved U8 0.16 mm to (112.9, 69.2)
Routing:
- net Net-(U6-Pad3): track 1.84 -> 2.39 mm
Other:
- net class Default: trace_width 0.254 -> 0.508

Commit message: Update
Parts:
- removed the REF** at (99.1, 53.3)
- removed the REF** at (88.9, 73.7)
- removed the REF** at (88.9, 38.1)
- removed the REF** at (88.9, 33.0)
- removed the REF** at (94.0, 38.1)
- removed the REF** at (104.1, 38.1)
- removed the REF** at (99.1, 38.1)
- removed the REF** at (58.4, 38.1)
- removed the REF** at (99.1, 68.6)
- removed the REF** at (109.2, 68.6)
- removed the REF** at (104.1, 68.6)
- removed the REF** at (104.1, 53.3)
- removed the REF** at (99.1, 73.7)
- removed the REF** at (104.1, 73.7)
- removed the REF** at (109.2, 73.7)
- removed the REF** at (58.4, 78.7)
- removed the REF** at (53.3, 78.7)
- removed the REF** at (48.3, 78.7)
- removed the REF** at (43.2, 78.7)
- removed the REF** at (43.2, 73.7)
- removed the REF** at (48.3, 73.7)
- removed the REF** at (53.3, 73.7)
- removed the REF** at (109.2, 53.3)
- removed the REF** at (58.4, 73.7)
- removed the REF** at (63.5, 73.7)
- removed the REF** at (63.5, 78.7)
- removed the REF** at (68.6, 73.7)
- removed the REF** at (68.6, 78.7)
- removed the REF** at (78.7, 78.7)
- removed the REF** at (78.7, 73.7)
- removed the REF** at (83.8, 73.7)
- removed the REF** at (83.8, 78.7)
- removed the REF** at (88.9, 83.8)
- removed the REF** at (114.3, 53.3)
- removed the REF** at (94.0, 83.8)
- removed the REF** at (99.1, 83.8)
- removed the REF** at (104.1, 83.8)
- removed the REF** at (109.2, 83.8)
- removed the REF** at (114.3, 83.8)
- removed the REF** at (119.4, 73.7)
- removed the REF** at (119.4, 68.6)
- removed the REF** at (119.4, 63.5)
- removed the REF** at (119.4, 58.4)
- removed the REF** at (119.4, 53.3)
- removed the REF** at (104.1, 43.2)
- removed the REF** at (94.0, 43.2)
- removed the REF** at (119.4, 43.2)
- removed the REF** at (119.4, 48.3)
- removed the REF** at (68.6, 63.5)
- removed the REF** at (63.5, 63.5)
- removed the REF** at (58.4, 63.5)
- removed the REF** at (38.1, 63.5)
- removed the REF** at (43.2, 63.5)
- removed the REF** at (53.3, 63.5)
- removed the REF** at (48.3, 63.5)
- removed the REF** at (99.1, 43.2)
- removed the REF** at (38.1, 38.1)
- removed the REF** at (88.9, 48.3)
- removed the REF** at (83.8, 48.3)
- removed the REF** at (78.7, 48.3)
- removed the REF** at (73.7, 48.3)
- removed the REF** at (114.3, 43.2)
- removed the REF** at (114.3, 38.1)
- removed the REF** at (114.3, 33.0)
- removed the REF** at (109.2, 33.0)
- removed the REF** at (104.1, 33.0)
- removed the REF** at (58.4, 43.2)
- removed the REF** at (99.1, 33.0)
- removed the REF** at (94.0, 33.0)
- removed the REF** at (58.4, 33.0)
- removed the REF** at (53.3, 33.0)
- removed the REF** at (48.3, 33.0)
- removed the REF** at (43.2, 33.0)
- removed the REF** at (38.1, 33.0)
- removed the REF** at (38.1, 43.2)
- removed the REF** at (43.2, 38.1)
- removed the REF** at (48.3, 38.1)
- removed the REF** at (43.2, 53.3)
- removed the REF** at (53.3, 38.1)
- removed the REF** at (43.2, 43.2)
- removed the REF** at (48.3, 43.2)
- removed the REF** at (53.3, 43.2)
- removed the REF** at (53.3, 53.3)
- removed the REF** at (48.3, 53.3)
- removed the REF** at (73.7, 33.0)
- removed the REF** at (78.7, 33.0)
- removed the REF** at (114.2, 48.3)
- removed the REF** at (63.5, 53.3)
- removed the REF** at (38.1, 48.3)
- removed TP10, TP11, TP12, TP13, TP14, TP9: TEST, Q2Footprint:PINTST
- added REF**: via-15mil, Q2Footprint:via-15mil, F.Cu at (75.7, 56.0)
- added REF**: via-15mil, Q2Footprint:via-15mil, F.Cu at (87.7, 34.0)
- added REF**: via-15mil, Q2Footprint:via-15mil, F.Cu at (37.7, 34.0)
- added REF**: via-15mil, Q2Footprint:via-15mil, F.Cu at (39.7, 34.0)
- added REF**: via-15mil, Q2Footprint:via-15mil, F.Cu at (41.7, 34.0)
- added REF**: via-15mil, Q2Footprint:via-15mil, F.Cu at (43.7, 34.0)
- added REF**: via-15mil, Q2Footprint:via-15mil, F.Cu at (45.7, 34.0)
- added REF**: via-15mil, Q2Footprint:via-15mil, F.Cu at (47.7, 34.0)
- added REF**: via-15mil, Q2Footprint:via-15mil, F.Cu at (39.7, 40.6)
- added REF**: via-15mil, Q2Footprint:via-15mil, F.Cu at (41.7, 40.6)
- added REF**: via-15mil, Q2Footprint:via-15mil, F.Cu at (43.7, 40.6)
- added REF**: via-15mil, Q2Footprint:via-15mil, F.Cu at (45.7, 40.6)
- added REF**: via-15mil, Q2Footprint:via-15mil, F.Cu at (89.7, 47.2)
- added REF**: via-15mil, Q2Footprint:via-15mil, F.Cu at (39.7, 45.0)
- added REF**: via-15mil, Q2Footprint:via-15mil, F.Cu at (43.7, 45.0)
- added REF**: via-15mil, Q2Footprint:via-15mil, F.Cu at (45.7, 45.0)
- added REF**: via-15mil, Q2Footprint:via-15mil, F.Cu at (47.7, 47.2)
- added REF**: via-15mil, Q2Footprint:via-15mil, F.Cu at (49.7, 47.2)
- added REF**: via-15mil, Q2Footprint:via-15mil, F.Cu at (49.7, 45.0)
- added REF**: via-15mil, Q2Footprint:via-15mil, F.Cu at (49.7, 42.8)
- added REF**: via-15mil, Q2Footprint:via-15mil, F.Cu at (49.7, 40.6)
- added REF**: via-15mil, Q2Footprint:via-15mil, F.Cu at (49.7, 36.2)
- added REF**: via-15mil, Q2Footprint:via-15mil, F.Cu at (49.7, 34.0)
- added REF**: via-15mil, Q2Footprint:via-15mil, F.Cu at (47.7, 45.0)
- added REF**: via-15mil, Q2Footprint:via-15mil, F.Cu at (91.7, 51.6)
- added REF**: via-15mil, Q2Footprint:via-15mil, F.Cu at (89.7, 51.6)
- added REF**: via-15mil, Q2Footprint:via-15mil, F.Cu at (87.7, 51.6)
- added REF**: via-15mil, Q2Footprint:via-15mil, F.Cu at (85.7, 51.6)
- added REF**: via-15mil, Q2Footprint:via-15mil, F.Cu at (83.7, 51.6)
- added REF**: via-15mil, Q2Footprint:via-15mil, F.Cu at (81.7, 51.6)
- added REF**: via-15mil, Q2Footprint:via-15mil, F.Cu at (79.7, 51.6)
- added REF**: via-15mil, Q2Footprint:via-15mil, F.Cu at (57.7, 53.8)
- added REF**: via-15mil, Q2Footprint:via-15mil, F.Cu at (71.7, 51.6)
- added REF**: via-15mil, Q2Footprint:via-15mil, F.Cu at (67.7, 51.6)
- added REF**: via-15mil, Q2Footprint:via-15mil, F.Cu at (69.7, 53.8)
- added REF**: via-15mil, Q2Footprint:via-15mil, F.Cu at (57.7, 51.6)
- added REF**: via-15mil, Q2Footprint:via-15mil, F.Cu at (37.7, 31.8)
- added REF**: via-15mil, Q2Footprint:via-15mil, F.Cu at (39.7, 31.8)
- added REF**: via-15mil, Q2Footprint:via-15mil, F.Cu at (41.7, 31.8)
- added REF**: via-15mil, Q2Footprint:via-15mil, F.Cu at (43.7, 31.8)
- added REF**: via-15mil, Q2Footprint:via-15mil, F.Cu at (45.7, 31.8)
- added REF**: via-15mil, Q2Footprint:via-15mil, F.Cu at (47.7, 31.8)
- added REF**: via-15mil, Q2Footprint:via-15mil, F.Cu at (49.7, 31.8)
- added REF**: via-15mil, Q2Footprint:via-15mil, F.Cu at (51.7, 31.8)
- added REF**: via-15mil, Q2Footprint:via-15mil, F.Cu at (53.7, 31.8)
- added REF**: via-15mil, Q2Footprint:via-15mil, F.Cu at (75.7, 49.4)
- added REF**: via-15mil, Q2Footprint:via-15mil, F.Cu at (55.7, 31.8)
- added REF**: via-15mil, Q2Footprint:via-15mil, F.Cu at (57.7, 31.8)
- added REF**: via-15mil, Q2Footprint:via-15mil, F.Cu at (59.7, 31.8)
- added REF**: via-15mil, Q2Footprint:via-15mil, F.Cu at (61.7, 31.8)
- added REF**: via-15mil, Q2Footprint:via-15mil, F.Cu at (63.7, 31.8)
- added REF**: via-15mil, Q2Footprint:via-15mil, F.Cu at (65.7, 31.8)
- added REF**: via-15mil, Q2Footprint:via-15mil, F.Cu at (67.7, 31.8)
- added REF**: via-15mil, Q2Footprint:via-15mil, F.Cu at (69.7, 31.8)
- added REF**: via-15mil, Q2Footprint:via-15mil, F.Cu at (71.7, 31.8)
- added REF**: via-15mil, Q2Footprint:via-15mil, F.Cu at (73.7, 31.8)
- added REF**: via-15mil, Q2Footprint:via-15mil, F.Cu at (73.7, 49.4)
- added REF**: via-15mil, Q2Footprint:via-15mil, F.Cu at (75.7, 31.8)
- added REF**: via-15mil, Q2Footprint:via-15mil, F.Cu at (77.7, 31.8)
- added REF**: via-15mil, Q2Footprint:via-15mil, F.Cu at (79.7, 31.8)
- added REF**: via-15mil, Q2Footprint:via-15mil, F.Cu at (81.7, 31.8)
- added REF**: via-15mil, Q2Footprint:via-15mil, F.Cu at (83.7, 31.8)
- added REF**: via-15mil, Q2Footprint:via-15mil, F.Cu at (85.7, 31.8)
- added REF**: via-15mil, Q2Footprint:via-15mil, F.Cu at (87.7, 31.8)
- added REF**: via-15mil, Q2Footprint:via-15mil, F.Cu at (71.7, 45.0)
- added REF**: via-15mil, Q2Footprint:via-15mil, F.Cu at (67.7, 45.1)
- added REF**: via-15mil, Q2Footprint:via-15mil, F.Cu at (59.7, 42.8)
- added REF**: via-15mil, Q2Footprint:via-15mil, F.Cu at (73.7, 45.0)
- added REF**: via-15mil, Q2Footprint:via-15mil, F.Cu at (57.7, 42.8)
- added REF**: via-15mil, Q2Footprint:via-15mil, F.Cu at (65.7, 42.8)
- added REF**: via-15mil, Q2Footprint:via-15mil, F.Cu at (63.7, 42.8)
- added REF**: via-15mil, Q2Footprint:via-15mil, F.Cu at (55.7, 51.6)
- added REF**: via-15mil, Q2Footprint:via-15mil, F.Cu at (55.7, 53.8)
- added REF**: via-15mil, Q2Footprint:via-15mil, F.Cu at (55.7, 56.0)
- added REF**: via-15mil, Q2Footprint:via-15mil, F.Cu at (53.7, 51.6)
- added REF**: via-15mil, Q2Footprint:via-15mil, F.Cu at (53.7, 53.8)
- added REF**: via-15mil, Q2Footprint:via-15mil, F.Cu at (53.7, 56.0)
- added REF**: via-15mil, Q2Footprint:via-15mil, F.Cu at (47.7, 51.6)
- added REF**: via-15mil, Q2Footprint:via-15mil, F.Cu at (93.7, 47.2)
- added REF**: via-15mil, Q2Footprint:via-15mil, F.Cu at (47.7, 53.8)
- added REF**: via-15mil, Q2Footprint:via-15mil, F.Cu at (47.7, 56.0)
- added REF**: via-15mil, Q2Footprint:via-15mil, F.Cu at (45.7, 56.0)
- added REF**: via-15mil, Q2Footprint:via-15mil, F.Cu at (45.7, 53.8)
- added REF**: via-15mil, Q2Footprint:via-15mil, F.Cu at (45.7, 51.6)
- added REF**: via-15mil, Q2Footprint:via-15mil, F.Cu at (43.7, 56.0)
- added REF**: via-15mil, Q2Footprint:via-15mil, F.Cu at (43.7, 53.8)
- added REF**: via-15mil, Q2Footprint:via-15mil, F.Cu at (43.7, 51.6)
- added REF**: via-15mil, Q2Footprint:via-15mil, F.Cu at (39.7, 51.6)
- added REF**: via-15mil, Q2Footprint:via-15mil, F.Cu at (39.7, 53.8)
- added REF**: via-15mil, Q2Footprint:via-15mil, F.Cu at (109.7, 49.4)
- added REF**: via-15mil, Q2Footprint:via-15mil, F.Cu at (39.7, 56.0)
- added REF**: via-15mil, Q2Footprint:via-15mil, F.Cu at (45.7, 49.4)
- added REF**: via-15mil, Q2Footprint:via-15mil, F.Cu at (43.7, 49.4)
- added REF**: via-15mil, Q2Footprint:via-15mil, F.Cu at (37.7, 49.4)
- added REF**: via-15mil, Q2Footprint:via-15mil, F.Cu at (37.7, 51.6)
- added REF**: via-15mil, Q2Footprint:via-15mil, F.Cu at (37.7, 53.8)
- added REF**: via-15mil, Q2Footprint:via-15mil, F.Cu at (37.7, 56.0)
- added REF**: via-15mil, Q2Footprint:via-15mil, F.Cu at (107.7, 40.6)
- added REF**: via-15mil, Q2Footprint:via-15mil, F.Cu at (105.7, 40.6)
- added REF**: via-15mil, Q2Footprint:via-15mil, F.Cu at (107.7, 42.8)
- added REF**: via-15mil, Q2Footprint:via-15mil, F.Cu at (113.7, 56.0)
- added REF**: via-15mil, Q2Footprint:via-15mil, F.Cu at (105.7, 42.8)
- added REF**: via-15mil, Q2Footprint:via-15mil, F.Cu at (107.7, 45.0)
- added REF**: via-15mil, Q2Footprint:via-15mil, F.Cu at (105.7, 45.0)
- added REF**: via-15mil, Q2Footprint:via-15mil, F.Cu at (107.7, 47.2)
- added REF**: via-15mil, Q2Footprint:via-15mil, F.Cu at (105.7, 47.2)
- added REF**: via-15mil, Q2Footprint:via-15mil, F.Cu at (105.7, 49.4)
- added REF**: via-15mil, Q2Footprint:via-15mil, F.Cu at (105.7, 51.6)
- added REF**: via-15mil, Q2Footprint:via-15mil, F.Cu at (105.7, 53.8)
- added REF**: via-15mil, Q2Footprint:via-15mil, F.Cu at (107.7, 53.8)
- added REF**: via-15mil, Q2Footprint:via-15mil, F.Cu at (107.7, 51.6)
- added REF**: via-15mil, Q2Footprint:via-15mil, F.Cu at (83.7, 38.4)
- added REF**: via-15mil, Q2Footprint:via-15mil, F.Cu at (119.7, 62.5)
- added REF**: via-15mil, Q2Footprint:via-15mil, F.Cu at (107.7, 49.4)
- added REF**: via-15mil, Q2Footprint:via-15mil, F.Cu at (111.7, 51.6)
- added REF**: via-15mil, Q2Footprint:via-15mil, F.Cu at (111.7, 49.4)
- added REF**: via-15mil, Q2Footprint:via-15mil, F.Cu at (93.7, 36.2)
- added REF**: via-15mil, Q2Footprint:via-15mil, F.Cu at (95.7, 36.2)
- added REF**: via-15mil, Q2Footprint:via-15mil, F.Cu at (97.7, 36.2)
- added REF**: via-15mil, Q2Footprint:via-15mil, F.Cu at (99.7, 36.2)
- added REF**: via-15mil, Q2Footprint:via-15mil, F.Cu at (101.7, 36.2)
- added REF**: via-15mil, Q2Footprint:via-15mil, F.Cu at (103.7, 36.2)
- added REF**: via-15mil, Q2Footprint:via-15mil, F.Cu at (105.7, 36.2)
- added REF**: via-15mil, Q2Footprint:via-15mil, F.Cu at (123.7, 62.5)
- added REF**: via-15mil, Q2Footprint:via-15mil, F.Cu at (107.7, 36.2)
- added REF**: via-15mil, Q2Footprint:via-15mil, F.Cu at (109.7, 36.2)
- added REF**: via-15mil, Q2Footprint:via-15mil, F.Cu at (111.7, 36.2)
- added REF**: via-15mil, Q2Footprint:via-15mil, F.Cu at (113.7, 36.2)
- added REF**: via-15mil, Q2Footprint:via-15mil, F.Cu at (115.7, 36.2)
- added REF**: via-15mil, Q2Footprint:via-15mil, F.Cu at (117.7, 36.2)
- added REF**: via-15mil, Q2Footprint:via-15mil, F.Cu at (119.7, 36.2)
- added REF**: via-15mil, Q2Footprint:via-15mil, F.Cu at (121.7, 36.2)
- added REF**: via-15mil, Q2Footprint:via-15mil, F.Cu at (123.7, 36.2)
- added REF**: via-15mil, Q2Footprint:via-15mil, F.Cu at (119.7, 42.8)
- added REF**: via-15mil, Q2Footprint:via-15mil, F.Cu at (121.7, 62.5)
- added REF**: via-15mil, Q2Footprint:via-15mil, F.Cu at (119.7, 45.0)
- added REF**: via-15mil, Q2Footprint:via-15mil, F.Cu at (111.7, 56.0)
- added REF**: via-15mil, Q2Footprint:via-15mil, F.Cu at (117.7, 49.4)
- added REF**: via-15mil, Q2Footprint:via-15mil, F.Cu at (119.7, 49.4)
- added REF**: via-15mil, Q2Footprint:via-15mil, F.Cu at (117.7, 51.6)
- added REF**: via-15mil, Q2Footprint:via-15mil, F.Cu at (119.7, 51.6)
- added REF**: via-15mil, Q2Footprint:via-15mil, F.Cu at (117.7, 53.8)
- added REF**: via-15mil, Q2Footprint:via-15mil, F.Cu at (119.7, 53.8)
- added REF**: via-15mil, Q2Footprint:via-15mil, F.Cu at (115.7, 38.4)
- added REF**: via-15mil, Q2Footprint:via-15mil, F.Cu at (117.7, 38.4)
- added REF**: via-15mil, Q2Footprint:via-15mil, F.Cu at (103.7, 71.3)
- added REF**: via-15mil, Q2Footprint:via-15mil, F.Cu at (119.7, 38.4)
- added REF**: via-15mil, Q2Footprint:via-15mil, F.Cu at (121.7, 38.4)
- added REF**: via-15mil, Q2Footprint:via-15mil, F.Cu at (89.7, 34.0)
- added REF**: via-15mil, Q2Footprint:via-15mil, F.Cu at (93.7, 34.0)
- added REF**: via-15mil, Q2Footprint:via-15mil, F.Cu at (95.7, 34.0)
- added REF**: via-15mil, Q2Footprint:via-15mil, F.Cu at (97.7, 34.0)
- added REF**: via-15mil, Q2Footprint:via-15mil, F.Cu at (99.7, 34.0)
- added REF**: via-15mil, Q2Footprint:via-15mil, F.Cu at (101.7, 34.0)
- added REF**: via-15mil, Q2Footprint:via-15mil, F.Cu at (103.7, 34.0)
- added REF**: via-15mil, Q2Footprint:via-15mil, F.Cu at (105.7, 34.0)
- added REF**: via-15mil, Q2Footprint:via-15mil, F.Cu at (103.7, 66.9)
- added REF**: via-15mil, Q2Footprint:via-15mil, F.Cu at (107.7, 34.0)
- added REF**: via-15mil, Q2Footprint:via-15mil, F.Cu at (109.7, 34.0)
- added REF**: via-15mil, Q2Footprint:via-15mil, F.Cu at (111.7, 34.0)
- added REF**: via-15mil, Q2Footprint:via-15mil, F.Cu at (113.7, 34.0)
- added REF**: via-15mil, Q2Footprint:via-15mil, F.Cu at (115.7, 34.0)
- added REF**: via-15mil, Q2Footprint:via-15mil, F.Cu at (117.7, 34.0)
- added REF**: via-15mil, Q2Footprint:via-15mil, F.Cu at (119.7, 34.0)
- added REF**: via-15mil, Q2Footprint:via-15mil, F.Cu at (121.7, 34.0)
- added REF**: via-15mil, Q2Footprint:via-15mil, F.Cu at (123.7, 34.0)
- added REF**: via-15mil, Q2Footprint:via-15mil, F.Cu at (89.7, 31.8)
- added REF**: via-15mil, Q2Footprint:via-15mil, F.Cu at (103.7, 69.1)
- added REF**: via-15mil, Q2Footprint:via-15mil, F.Cu at (91.7, 31.8)
- added REF**: via-15mil, Q2Footprint:via-15mil, F.Cu at (93.7, 31.8)
- added REF**: via-15mil, Q2Footprint:via-15mil, F.Cu at (95.7, 31.8)
- added REF**: via-15mil, Q2Footprint:via-15mil, F.Cu at (97.7, 31.8)
- added REF**: via-15mil, Q2Footprint:via-15mil, F.Cu at (99.7, 31.8)
- added REF**: via-15mil, Q2Footprint:via-15mil, F.Cu at (101.7, 31.8)
- added REF**: via-15mil, Q2Footprint:via-15mil, F.Cu at (103.7, 31.8)
- added REF**: via-15mil, Q2Footprint:via-15mil, F.Cu at (105.7, 31.8)
- added REF**: via-15mil, Q2Footprint:via-15mil, F.Cu at (107.7, 31.8)
- added REF**: via-15mil, Q2Footprint:via-15mil, F.Cu at (109.7, 31.8)
- added REF**: via-15mil, Q2Footprint:via-15mil, F.Cu at (115.7, 66.9)
- added REF**: via-15mil, Q2Footprint:via-15mil, F.Cu at (111.7, 31.8)
- added REF**: via-15mil, Q2Footprint:via-15mil, F.Cu at (113.7, 31.8)
- added REF**: via-15mil, Q2Footprint:via-15mil, F.Cu at (115.7, 31.8)
- added REF**: via-15mil, Q2Footprint:via-15mil, F.Cu at (117.7, 31.8)
- added REF**: via-15mil, Q2Footprint:via-15mil, F.Cu at (119.7, 31.8)
- added REF**: via-15mil, Q2Footprint:via-15mil, F.Cu at (121.7, 31.8)
- added REF**: via-15mil, Q2Footprint:via-15mil, F.Cu at (123.7, 31.8)
- added REF**: via-15mil, Q2Footprint:via-15mil, F.Cu at (123.7, 38.4)
- added REF**: via-15mil, Q2Footprint:via-15mil, F.Cu at (123.7, 42.8)
- added REF**: via-15mil, Q2Footprint:via-15mil, F.Cu at (123.7, 45.0)
- added REF**: via-15mil, Q2Footprint:via-15mil, F.Cu at (115.7, 62.5)
- added REF**: via-15mil, Q2Footprint:via-15mil, F.Cu at (123.7, 47.2)
- added REF**: via-15mil, Q2Footprint:via-15mil, F.Cu at (123.7, 49.4)
- added REF**: via-15mil, Q2Footprint:via-15mil, F.Cu at (123.7, 51.6)
- added REF**: via-15mil, Q2Footprint:via-15mil, F.Cu at (123.7, 53.8)
- added REF**: via-15mil, Q2Footprint:via-15mil, F.Cu at (127.7, 40.6)
- added REF**: via-15mil, Q2Footprint:via-15mil, F.Cu at (127.7, 42.8)
- added REF**: via-15mil, Q2Footprint:via-15mil, F.Cu at (127.7, 45.0)
- added REF**: via-15mil, Q2Footprint:via-15mil, F.Cu at (127.7, 47.2)
- added REF**: via-15mil, Q2Footprint:via-15mil, F.Cu at (127.7, 49.4)
- added REF**: via-15mil, Q2Footprint:via-15mil, F.Cu at (127.7, 51.6)
- added REF**: via-15mil, Q2Footprint:via-15mil, F.Cu at (97.7, 71.3)
- added REF**: via-15mil, Q2Footprint:via-15mil, F.Cu at (127.7, 53.8)
- added REF**: via-15mil, Q2Footprint:via-15mil, F.Cu at (127.7, 56.0)
- added REF**: via-15mil, Q2Footprint:via-15mil, F.Cu at (123.7, 56.0)
- added REF**: via-15mil, Q2Footprint:via-15mil, F.Cu at (117.7, 56.0)
- added REF**: via-15mil, Q2Footprint:via-15mil, F.Cu at (127.7, 66.9)
- added REF**: via-15mil, Q2Footprint:via-15mil, F.Cu at (125.7, 66.9)
- added REF**: via-15mil, Q2Footprint:via-15mil, F.Cu at (123.7, 66.9)
- added REF**: via-15mil, Q2Footprint:via-15mil, F.Cu at (121.7, 66.9)
- added REF**: via-15mil, Q2Footprint:via-15mil, F.Cu at (119.7, 66.9)
- added REF**: via-15mil, Q2Footprint:via-15mil, F.Cu at (117.7, 66.9)
- added REF**: via-15mil, Q2Footprint:via-15mil, F.Cu at (95.7, 71.3)
- added REF**: via-15mil, Q2Footprint:via-15mil, F.Cu at (117.7, 62.5)
- added REF**: via-15mil, Q2Footprint:via-15mil, F.Cu at (113.7, 62.5)
- added REF**: via-15mil, Q2Footprint:via-15mil, F.Cu at (111.7, 66.9)
- added REF**: via-15mil, Q2Footprint:via-15mil, F.Cu at (111.7, 64.7)
- added REF**: via-15mil, Q2Footprint:via-15mil, F.Cu at (111.7, 62.5)
- added REF**: via-15mil, Q2Footprint:via-15mil, F.Cu at (103.7, 64.7)
- added REF**: via-15mil, Q2Footprint:via-15mil, F.Cu at (103.7, 62.5)
- added REF**: via-15mil, Q2Footprint:via-15mil, F.Cu at (99.7, 66.9)
- added REF**: via-15mil, Q2Footprint:via-15mil, F.Cu at (99.7, 64.7)
- added REF**: via-15mil, Q2Footprint:via-15mil, F.Cu at (99.7, 62.5)
- added REF**: via-15mil, Q2Footprint:via-15mil, F.Cu at (83.7, 36.2)
- added REF**: via-15mil, Q2Footprint:via-15mil, F.Cu at (87.7, 73.5)
- added REF**: via-15mil, Q2Footprint:via-15mil, F.Cu at (101.7, 62.5)
- added REF**: via-15mil, Q2Footprint:via-15mil, F.Cu at (101.7, 64.7)
- added REF** (x2): via-15mil, Q2Footprint:via-15mil, F.Cu at (121.7, 69.1)
- added REF** (x2): via-15mil, Q2Footprint:via-15mil, F.Cu at (119.7, 69.1)
- added REF** (x2): via-15mil, Q2Footprint:via-15mil, F.Cu at (117.7, 69.1)
- added REF** (x2): via-15mil, Q2Footprint:via-15mil, F.Cu at (115.7, 69.1)
- added REF**: via-15mil, Q2Footprint:via-15mil, F.Cu at (123.7, 71.0)
- added REF**: via-15mil, Q2Footprint:via-15mil, F.Cu at (121.7, 71.0)
- added REF**: via-15mil, Q2Footprint:via-15mil, F.Cu at (119.7, 71.0)
- added REF**: via-15mil, Q2Footprint:via-15mil, F.Cu at (117.7, 71.0)
- added REF**: via-15mil, Q2Footprint:via-15mil, F.Cu at (89.7, 73.5)
- added REF**: via-15mil, Q2Footprint:via-15mil, F.Cu at (115.7, 71.0)
- added REF**: via-15mil, Q2Footprint:via-15mil, F.Cu at (101.7, 66.9)
- added REF**: via-15mil, Q2Footprint:via-15mil, F.Cu at (101.7, 69.1)
- added REF**: via-15mil, Q2Footprint:via-15mil, F.Cu at (105.7, 66.9)
- added REF**: via-15mil, Q2Footprint:via-15mil, F.Cu at (105.7, 69.1)
- added REF**: via-15mil, Q2Footprint:via-15mil, F.Cu at (111.7, 69.1)
- added REF**: via-15mil, Q2Footprint:via-15mil, F.Cu at (123.7, 69.1)
- added REF**: via-15mil, Q2Footprint:via-15mil, F.Cu at (91.7, 73.5)
- added REF**: via-15mil, Q2Footprint:via-15mil, F.Cu at (123.7, 73.5)
- added REF**: via-15mil, Q2Footprint:via-15mil, F.Cu at (121.7, 73.5)
- added REF**: via-15mil, Q2Footprint:via-15mil, F.Cu at (119.7, 73.5)
- added REF**: via-15mil, Q2Footprint:via-15mil, F.Cu at (117.7, 73.5)
- added REF**: via-15mil, Q2Footprint:via-15mil, F.Cu at (115.7, 73.5)
- added REF**: via-15mil, Q2Footprint:via-15mil, F.Cu at (113.7, 73.5)
- added REF**: via-15mil, Q2Footprint:via-15mil, F.Cu at (111.7, 73.5)
- added REF**: via-15mil, Q2Footprint:via-15mil, F.Cu at (109.7, 73.5)
- added REF**: via-15mil, Q2Footprint:via-15mil, F.Cu at (107.7, 73.5)
- added REF**: via-15mil, Q2Footprint:via-15mil, F.Cu at (93.7, 73.5)
- added REF**: via-15mil, Q2Footprint:via-15mil, F.Cu at (105.7, 73.5)
- added REF**: via-15mil, Q2Footprint:via-15mil, F.Cu at (103.7, 73.5)
- added REF**: via-15mil, Q2Footprint:via-15mil, F.Cu at (101.7, 73.5)
- added REF**: via-15mil, Q2Footprint:via-15mil, F.Cu at (99.7, 73.5)
- added REF**: via-15mil, Q2Footprint:via-15mil, F.Cu at (97.7, 73.5)
- added REF**: via-15mil, Q2Footprint:via-15mil, F.Cu at (127.7, 77.9)
- added REF**: via-15mil, Q2Footprint:via-15mil, F.Cu at (125.7, 77.9)
- added REF**: via-15mil, Q2Footprint:via-15mil, F.Cu at (123.7, 77.9)
- added REF**: via-15mil, Q2Footprint:via-15mil, F.Cu at (121.7, 77.9)
- added REF**: via-15mil, Q2Footprint:via-15mil, F.Cu at (119.7, 77.9)
- added REF**: via-15mil, Q2Footprint:via-15mil, F.Cu at (95.7, 73.5)
- added REF**: via-15mil, Q2Footprint:via-15mil, F.Cu at (117.7, 77.9)
- added REF**: via-15mil, Q2Footprint:via-15mil, F.Cu at (115.7, 77.9)
- added REF**: via-15mil, Q2Footprint:via-15mil, F.Cu at (113.7, 77.9)
- added REF**: via-15mil, Q2Footprint:via-15mil, F.Cu at (111.7, 77.9)
- added REF**: via-15mil, Q2Footprint:via-15mil, F.Cu at (109.7, 77.9)
- added REF**: via-15mil, Q2Footprint:via-15mil, F.Cu at (107.7, 77.9)
- added REF**: via-15mil, Q2Footprint:via-15mil, F.Cu at (105.7, 77.9)
- added REF**: via-15mil, Q2Footprint:via-15mil, F.Cu at (103.7, 77.9)
- added REF**: via-15mil, Q2Footprint:via-15mil, F.Cu at (101.7, 77.9)
- added REF**: via-15mil, Q2Footprint:via-15mil, F.Cu at (99.7, 77.9)
- added REF**: via-15mil, Q2Footprint:via-15mil, F.Cu at (95.7, 66.9)
- added REF**: via-15mil, Q2Footprint:via-15mil, F.Cu at (97.7, 77.9)
- added REF**: via-15mil, Q2Footprint:via-15mil, F.Cu at (95.7, 77.9)
- added REF**: via-15mil, Q2Footprint:via-15mil, F.Cu at (93.7, 77.9)
- added REF**: via-15mil, Q2Footprint:via-15mil, F.Cu at (91.7, 77.9)
- added REF**: via-15mil, Q2Footprint:via-15mil, F.Cu at (89.7, 77.9)
- added REF**: via-15mil, Q2Footprint:via-15mil, F.Cu at (123.7, 75.7)
- added REF**: via-15mil, Q2Footprint:via-15mil, F.Cu at (121.7, 75.7)
- added REF**: via-15mil, Q2Footprint:via-15mil, F.Cu at (119.7, 75.7)
- added REF**: via-15mil, Q2Footprint:via-15mil, F.Cu at (117.7, 75.7)
- added REF**: via-15mil, Q2Footprint:via-15mil, F.Cu at (115.7, 75.7)
- added REF**: via-15mil, Q2Footprint:via-15mil, F.Cu at (97.7, 66.9)
- added REF**: via-15mil, Q2Footprint:via-15mil, F.Cu at (113.7, 75.7)
- added REF**: via-15mil, Q2Footprint:via-15mil, F.Cu at (111.7, 75.7)
- added REF**: via-15mil, Q2Footprint:via-15mil, F.Cu at (109.7, 75.7)
- added REF**: via-15mil, Q2Footprint:via-15mil, F.Cu at (107.7, 75.7)
- added REF**: via-15mil, Q2Footprint:via-15mil, F.Cu at (105.7, 75.7)
- added REF**: via-15mil, Q2Footprint:via-15mil, F.Cu at (103.7, 75.7)
- added REF**: via-15mil, Q2Footprint:via-15mil, F.Cu at (101.7, 75.7)
- added REF**: via-15mil, Q2Footprint:via-15mil, F.Cu at (99.7, 75.7)
- added REF**: via-15mil, Q2Footprint:via-15mil, F.Cu at (97.7, 75.7)
- added REF**: via-15mil, Q2Footprint:via-15mil, F.Cu at (95.7, 75.7)
- added REF**: via-15mil, Q2Footprint:via-15mil, F.Cu at (95.7, 64.7)
- added REF**: via-15mil, Q2Footprint:via-15mil, F.Cu at (93.7, 75.7)
- added REF**: via-15mil, Q2Footprint:via-15mil, F.Cu at (91.7, 75.7)
- added REF**: via-15mil, Q2Footprint:via-15mil, F.Cu at (89.7, 75.7)
- added REF**: via-15mil, Q2Footprint:via-15mil, F.Cu at (85.7, 73.5)
- added REF**: via-15mil, Q2Footprint:via-15mil, F.Cu at (83.7, 73.5)
- added REF**: via-15mil, Q2Footprint:via-15mil, F.Cu at (85.7, 62.5)
- added REF**: via-15mil, Q2Footprint:via-15mil, F.Cu at (83.7, 62.5)
- added REF**: via-15mil, Q2Footprint:via-15mil, F.Cu at (93.7, 71.3)
- added REF**: via-15mil, Q2Footprint:via-15mil, F.Cu at (91.7, 71.3)
- added REF**: via-15mil, Q2Footprint:via-15mil, F.Cu at (89.7, 71.3)
- added REF**: via-15mil, Q2Footprint:via-15mil, F.Cu at (97.7, 64.7)
- added REF**: via-15mil, Q2Footprint:via-15mil, F.Cu at (93.7, 69.1)
- added REF**: via-15mil, Q2Footprint:via-15mil, F.Cu at (91.7, 69.1)
- added REF**: via-15mil, Q2Footprint:via-15mil, F.Cu at (89.7, 69.1)
- added REF**: via-15mil, Q2Footprint:via-15mil, F.Cu at (93.7, 66.9)
- added REF**: via-15mil, Q2Footprint:via-15mil, F.Cu at (91.7, 66.9)
- added REF**: via-15mil, Q2Footprint:via-15mil, F.Cu at (89.7, 66.9)
- added REF**: via-15mil, Q2Footprint:via-15mil, F.Cu at (93.7, 64.7)
- added REF**: via-15mil, Q2Footprint:via-15mil, F.Cu at (91.7, 64.7)
- added REF**: via-15mil, Q2Footprint:via-15mil, F.Cu at (89.7, 64.7)
- added REF**: via-15mil, Q2Footprint:via-15mil, F.Cu at (83.7, 77.9)
- added REF**: via-15mil, Q2Footprint:via-15mil, F.Cu at (95.7, 62.5)
- added REF**: via-15mil, Q2Footprint:via-15mil, F.Cu at (85.7, 77.9)
- added REF**: via-15mil, Q2Footprint:via-15mil, F.Cu at (83.7, 75.7)
- added REF**: via-15mil, Q2Footprint:via-15mil, F.Cu at (85.7, 75.7)
- added REF**: via-15mil, Q2Footprint:via-15mil, F.Cu at (87.7, 77.9)
- added REF**: via-15mil, Q2Footprint:via-15mil, F.Cu at (87.7, 75.7)
- added REF**: via-15mil, Q2Footprint:via-15mil, F.Cu at (87.7, 71.3)
- added REF**: via-15mil, Q2Footprint:via-15mil, F.Cu at (87.7, 69.1)
- added REF**: via-15mil, Q2Footprint:via-15mil, F.Cu at (87.7, 66.9)
- added REF**: via-15mil, Q2Footprint:via-15mil, F.Cu at (87.7, 64.7)
- added REF**: via-15mil, Q2Footprint:via-15mil, F.Cu at (77.7, 64.7)
- added REF**: via-15mil, Q2Footprint:via-15mil, F.Cu at (81.7, 36.2)
- added REF**: via-15mil, Q2Footprint:via-15mil, F.Cu at (97.7, 62.5)
- added REF**: via-15mil, Q2Footprint:via-15mil, F.Cu at (75.7, 64.7)
- added REF**: via-15mil, Q2Footprint:via-15mil, F.Cu at (73.7, 64.7)
- added REF**: via-15mil, Q2Footprint:via-15mil, F.Cu at (71.7, 64.7)
- added REF**: via-15mil, Q2Footprint:via-15mil, F.Cu at (69.7, 64.7)
- added REF**: via-15mil, Q2Footprint:via-15mil, F.Cu at (67.7, 64.7)
- added REF**: via-15mil, Q2Footprint:via-15mil, F.Cu at (65.7, 64.7)
- added REF**: via-15mil, Q2Footprint:via-15mil, F.Cu at (63.7, 64.7)
- added REF**: via-15mil, Q2Footprint:via-15mil, F.Cu at (45.7, 77.9)
- added REF**: via-15mil, Q2Footprint:via-15mil, F.Cu at (43.7, 77.9)
- added REF**: via-15mil, Q2Footprint:via-15mil, F.Cu at (41.7, 77.9)
- added REF**: via-15mil, Q2Footprint:via-15mil, F.Cu at (89.7, 62.5)
- added REF**: via-15mil, Q2Footprint:via-15mil, F.Cu at (39.7, 77.9)
- added REF**: via-15mil, Q2Footprint:via-15mil, F.Cu at (77.7, 75.7)
- added REF**: via-15mil, Q2Footprint:via-15mil, F.Cu at (75.7, 75.7)
- added REF**: via-15mil, Q2Footprint:via-15mil, F.Cu at (73.7, 75.7)
- added REF**: via-15mil, Q2Footprint:via-15mil, F.Cu at (71.7, 75.7)
- added REF**: via-15mil, Q2Footprint:via-15mil, F.Cu at (69.7, 75.7)
- added REF**: via-15mil, Q2Footprint:via-15mil, F.Cu at (67.7, 75.7)
- added REF**: via-15mil, Q2Footprint:via-15mil, F.Cu at (65.7, 75.7)
- added REF**: via-15mil, Q2Footprint:via-15mil, F.Cu at (63.7, 75.7)
- added REF**: via-15mil, Q2Footprint:via-15mil, F.Cu at (61.7, 75.7)
- added REF**: via-15mil, Q2Footprint:via-15mil, F.Cu at (87.7, 62.5)
- added REF**: via-15mil, Q2Footprint:via-15mil, F.Cu at (59.7, 75.7)
- added REF**: via-15mil, Q2Footprint:via-15mil, F.Cu at (57.7, 75.7)
- added REF**: via-15mil, Q2Footprint:via-15mil, F.Cu at (55.7, 75.7)
- added REF**: via-15mil, Q2Footprint:via-15mil, F.Cu at (53.7, 75.7)
- added REF**: via-15mil, Q2Footprint:via-15mil, F.Cu at (51.7, 75.7)
- added REF**: via-15mil, Q2Footprint:via-15mil, F.Cu at (49.7, 75.7)
- added REF**: via-15mil, Q2Footprint:via-15mil, F.Cu at (47.7, 75.7)
- added REF**: via-15mil, Q2Footprint:via-15mil, F.Cu at (45.7, 75.7)
- added REF**: via-15mil, Q2Footprint:via-15mil, F.Cu at (43.7, 75.7)
- added REF**: via-15mil, Q2Footprint:via-15mil, F.Cu at (41.7, 75.7)
- added REF**: via-15mil, Q2Footprint:via-15mil, F.Cu at (83.7, 71.3)
- added REF**: via-15mil, Q2Footprint:via-15mil, F.Cu at (39.7, 75.7)
- added REF**: via-15mil, Q2Footprint:via-15mil, F.Cu at (77.7, 73.5)
- added REF**: via-15mil, Q2Footprint:via-15mil, F.Cu at (75.7, 73.5)
- added REF**: via-15mil, Q2Footprint:via-15mil, F.Cu at (73.7, 73.5)
- added REF**: via-15mil, Q2Footprint:via-15mil, F.Cu at (71.7, 73.5)
- added REF**: via-15mil, Q2Footprint:via-15mil, F.Cu at (69.7, 73.5)
- added REF**: via-15mil, Q2Footprint:via-15mil, F.Cu at (67.7, 73.5)
- added REF**: via-15mil, Q2Footprint:via-15mil, F.Cu at (65.7, 73.5)
- added REF**: via-15mil, Q2Footprint:via-15mil, F.Cu at (63.7, 73.5)
- added REF**: via-15mil, Q2Footprint:via-15mil, F.Cu at (61.7, 73.5)
- added REF**: via-15mil, Q2Footprint:via-15mil, F.Cu at (85.7, 71.3)
- added REF**: via-15mil, Q2Footprint:via-15mil, F.Cu at (59.7, 73.5)
- added REF**: via-15mil, Q2Footprint:via-15mil, F.Cu at (57.7, 73.5)
- added REF**: via-15mil, Q2Footprint:via-15mil, F.Cu at (55.7, 73.5)
- added REF**: via-15mil, Q2Footprint:via-15mil, F.Cu at (53.7, 73.5)
- added REF**: via-15mil, Q2Footprint:via-15mil, F.Cu at (51.7, 73.5)
- added REF**: via-15mil, Q2Footprint:via-15mil, F.Cu at (49.7, 73.5)
- added REF**: via-15mil, Q2Footprint:via-15mil, F.Cu at (47.7, 73.5)
- added REF**: via-15mil, Q2Footprint:via-15mil, F.Cu at (45.7, 73.5)
- added REF**: via-15mil, Q2Footprint:via-15mil, F.Cu at (43.7, 73.5)
- added REF**: via-15mil, Q2Footprint:via-15mil, F.Cu at (41.7, 73.5)
- added REF**: via-15mil, Q2Footprint:via-15mil, F.Cu at (83.7, 69.1)
- added REF**: via-15mil, Q2Footprint:via-15mil, F.Cu at (39.7, 73.5)
- added REF**: via-15mil, Q2Footprint:via-15mil, F.Cu at (77.7, 71.3)
- added REF**: via-15mil, Q2Footprint:via-15mil, F.Cu at (75.7, 71.3)
- added REF**: via-15mil, Q2Footprint:via-15mil, F.Cu at (73.7, 71.3)
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Connections:
- C8 pad 1: Net-(C8-Pad1) -> /+5V
- C8 pad 2: /+5V -> GND
- TP7 pad 1: Net-(C7-Pad2) -> Net-(C13-Pad1)
- TP8 pad 1: Net-(C12-Pad1) -> Net-(C14-Pad2)
- U2 pad 32: Net-(U2-Pad32) -> /+5V
- U7 pad : (no net) -> GND
- U7 pad 3: Net-(C8-Pad1) -> /+5V
Routing:
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Other:
- board size 86 x 55 mm -> 94 x 49 mm
- net class Default: trace_width 0.508 -> 0.572
- net class Fat added: clearance 0.1524, trace_width 1.08408, via_dia 0.762, via_drill 0.381
- net class LNA added: clearance 0.1524, trace_width 1.08408, via_dia 0.762, via_drill 0.381
- rule trace_min: 0.1524 -> 0.1778
- board text added: "UC Davis EEC 134"

Commit message: Update
Parts:
- added REF**: via-15mil, Q2Footprint:via-15mil, F.Cu at (100.8, 42.2)
- added REF**: via-15mil, Q2Footprint:via-15mil, F.Cu at (119.7, 63.8)
- added REF**: via-15mil, Q2Footprint:via-15mil, F.Cu at (113.3, 68.9)
- added REF**: via-15mil, Q2Footprint:via-15mil, F.Cu at (123.6, 40.0)
- added REF**: via-15mil, Q2Footprint:via-15mil, F.Cu at (119.9, 40.0)
- added REF**: via-15mil, Q2Footprint:via-15mil, F.Cu at (117.1, 48.2)
- added REF**: via-15mil, Q2Footprint:via-15mil, F.Cu at (117.1, 45.0)
- added REF**: via-15mil, Q2Footprint:via-15mil, F.Cu at (92.8, 45.5)
- added REF**: via-15mil, Q2Footprint:via-15mil, F.Cu at (110.8, 45.4)
- added REF**: via-15mil, Q2Footprint:via-15mil, F.Cu at (110.8, 42.6)
- added REF**: via-15mil, Q2Footprint:via-15mil, F.Cu at (110.8, 39.9)
- added REF**: via-15mil, Q2Footprint:via-15mil, F.Cu at (99.0, 43.4)
- added REF**: via-15mil, Q2Footprint:via-15mil, F.Cu at (99.3, 48.1)
- added REF**: via-15mil, Q2Footprint:via-15mil, F.Cu at (99.3, 44.8)
- added REF**: via-15mil, Q2Footprint:via-15mil, F.Cu at (101.8, 44.7)
- added REF**: via-15mil, Q2Footprint:via-15mil, F.Cu at (102.5, 47.2)
- added REF**: via-15mil, Q2Footprint:via-15mil, F.Cu at (110.4, 37.5)
- added REF**: via-15mil, Q2Footprint:via-15mil, F.Cu at (108.5, 37.5)
- added REF**: via-15mil, Q2Footprint:via-15mil, F.Cu at (92.9, 42.3)
- added REF**: via-15mil, Q2Footprint:via-15mil, F.Cu at (94.5, 42.3)
- added REF**: via-15mil, Q2Footprint:via-15mil, F.Cu at (95.8, 40.1)
- added REF**: via-15mil, Q2Footprint:via-15mil, F.Cu at (93.7, 40.1)
- added REF**: via-15mil, Q2Footprint:via-15mil, F.Cu at (118.7, 42.2)
- added REF**: via-15mil, Q2Footprint:via-15mil, F.Cu at (116.9, 43.4)
- added REF**: via-15mil, Q2Footprint:via-15mil, F.Cu at (113.4, 70.9)
- added REF**: via-15mil, Q2Footprint:via-15mil, F.Cu at (123.7, 65.1)
- added REF**: via-15mil, Q2Footprint:via-15mil, F.Cu at (121.7, 63.8)
- added REF**: via-15mil, Q2Footprint:via-15mil, F.Cu at (113.3, 66.9)
- added REF**: via-15mil, Q2Footprint:via-15mil, F.Cu at (98.5, 70.0)
- moved REF** 1.91 mm to (116.1, 65.0)
Routing:
- net Net-(U8-Pad8): track 5.65 -> 4.85 mm
- net Net-(U10-Pad5): track 3.09 -> 2.45 mm

Commit message: Update
Parts:
- removed the REF** at (93.7, 38.4)
- removed the REF** at (93.7, 36.2)
- removed the REF** at (93.7, 34.0)
- removed the REF** at (93.7, 31.8)
- removed the REF** at (127.7, 66.9)
- removed the REF** at (119.7, 69.1) (x2)
- removed the REF** at (117.7, 69.1) (x2)
- removed the REF** at (115.7, 69.1)
- removed the REF** at (123.7, 71.0)
- removed the REF** at (121.7, 71.0)
- removed the REF** at (119.7, 71.0)
- removed the REF** at (117.7, 71.0)
- removed the REF** at (123.7, 69.1)
- removed the REF** at (123.7, 73.5)
- removed the REF** at (121.7, 73.5)
- removed the REF** at (119.7, 73.5)
- removed the REF** at (117.7, 73.5)
- removed the REF** at (123.7, 75.7)
- removed the REF** at (119.7, 75.7)
- removed the REF** at (117.7, 75.7)
- removed the REF** at (77.7, 64.7)
- removed the REF** at (75.7, 64.7)
- removed the REF** at (73.7, 64.7)
- removed the REF** at (45.7, 77.9)
- removed the REF** at (43.7, 77.9)
- removed the REF** at (41.7, 77.9)
- removed the REF** at (39.7, 77.9)
- removed the REF** at (73.7, 75.7)
- removed the REF** at (73.7, 73.5)
- removed the REF** at (73.7, 71.3)
- removed the REF** at (73.7, 69.1)
- removed the REF** at (73.7, 66.9)
- removed the REF** at (47.7, 64.7)
- removed the REF** at (43.7, 64.7)
- removed the REF** at (45.7, 62.5)
- removed the REF** at (43.7, 62.5)
- removed the REF** at (41.7, 62.5)
- removed the REF** at (39.7, 62.5)
- removed the REF** at (43.7, 60.3)
- removed the REF** at (41.7, 60.3)
- removed the REF** at (41.7, 58.2)
- added REF**: via-15mil, Q2Footprint:via-15mil, F.Cu at (55.7, 64.7)
- added REF**: via-15mil, Q2Footprint:via-15mil, F.Cu at (75.7, 62.5)
- added REF**: via-15mil, Q2Footprint:via-15mil, F.Cu at (77.7, 77.9)
- added REF**: via-15mil, Q2Footprint:via-15mil, F.Cu at (77.7, 62.5)
- added REF**: via-15mil, Q2Footprint:via-15mil, F.Cu at (57.7, 64.7)
- added REF**: via-15mil, Q2Footprint:via-15mil, F.Cu at (81.7, 77.9)
- added REF**: via-15mil, Q2Footprint:via-15mil, F.Cu at (81.7, 75.7)
- added REF**: via-15mil, Q2Footprint:via-15mil, F.Cu at (81.7, 73.5)
- added REF**: via-15mil, Q2Footprint:via-15mil, F.Cu at (81.7, 71.3)
- added REF**: via-15mil, Q2Footprint:via-15mil, F.Cu at (81.7, 69.1)
- added REF**: via-15mil, Q2Footprint:via-15mil, F.Cu at (81.7, 64.7)
- added REF**: via-15mil, Q2Footprint:via-15mil, F.Cu at (81.7, 62.5)
- added REF**: via-15mil, Q2Footprint:via-15mil, F.Cu at (79.7, 77.9)
- added REF**: via-15mil, Q2Footprint:via-15mil, F.Cu at (79.7, 75.7)
- added REF**: via-15mil, Q2Footprint:via-15mil, F.Cu at (79.7, 73.5)
- added REF**: via-15mil, Q2Footprint:via-15mil, F.Cu at (59.7, 64.7)
- added REF**: via-15mil, Q2Footprint:via-15mil, F.Cu at (79.7, 71.3)
- added REF**: via-15mil, Q2Footprint:via-15mil, F.Cu at (79.7, 69.1)
- added REF**: via-15mil, Q2Footprint:via-15mil, F.Cu at (79.7, 66.9)
- added REF**: via-15mil, Q2Footprint:via-15mil, F.Cu at (79.7, 62.5)
- added REF**: via-15mil, Q2Footprint:via-15mil, F.Cu at (127.7, 60.4)
- added REF**: via-15mil, Q2Footprint:via-15mil, F.Cu at (127.7, 58.2)
- added REF**: via-15mil, Q2Footprint:via-15mil, F.Cu at (125.7, 73.5)
- added REF**: via-15mil, Q2Footprint:via-15mil, F.Cu at (125.7, 71.3)
- added REF**: via-15mil, Q2Footprint:via-15mil, F.Cu at (127.7, 73.5)
- added REF**: via-15mil, Q2Footprint:via-15mil, F.Cu at (127.7, 71.3)
- added REF**: via-15mil, Q2Footprint:via-15mil, F.Cu at (61.7, 64.7)
- added REF**: via-15mil, Q2Footprint:via-15mil, F.Cu at (45.7, 60.3)
- added REF**: via-15mil, Q2Footprint:via-15mil, F.Cu at (127.7, 36.2)
- added REF**: via-15mil, Q2Footprint:via-15mil, F.Cu at (125.7, 36.2)
- added REF**: via-15mil, Q2Footprint:via-15mil, F.Cu at (127.7, 34.0)
- added REF**: via-15mil, Q2Footprint:via-15mil, F.Cu at (125.7, 34.0)
- added REF**: via-15mil, Q2Footprint:via-15mil, F.Cu at (91.7, 36.2)
- added REF**: via-15mil, Q2Footprint:via-15mil, F.Cu at (91.7, 34.0)
- added REF**: via-15mil, Q2Footprint:via-15mil, F.Cu at (75.7, 77.9)
- added TP9: TEST, Q2Footprint:PINTST, F.Cu at (79.4, 65.2)
- U11: footprint Q2Footprint:SMA -> Q2Footprint:SMA_Vertical
- moved TP7 55.3 mm to (76.7, 76.9)
- moved U3 36.0 mm to (93.7, 31.0), turned to 180 degrees
- moved U2 6.70 mm to (75.2, 69.8)
- moved U11 3.81 mm to (121.2, 72.1), turned to 0 degrees
- moved C13 2.56 mm to (128.7, 65.0), turned to 90 degrees
- moved C3 1.89 mm to (92.5, 37.7), turned to 0 degrees
- moved R7 0.13 mm to (86.1, 37.3)
- moved TP6 0.08 mm to (86.1, 33.4)
Routing:
- net Net-(C3-Pad2): track 36.1 -> 4.49 mm
- net Net-(C13-Pad1): track 69.4 -> 97.5 mm
- net Net-(U10-Pad1): track 27.2 -> 9.68 mm
- net Net-(TP9-Pad1): track 4.83 -> 11.5 mm
- net /+5V: track 203.3 -> 205.9 mm
- net Net-(U8-Pad8): track 4.85 -> 3.04 mm
Other:
- board text removed: "UC Davis EEC 134"
