File: Q2.sch (KiCad schematic (older format))
At the start: 72 parts, among them U1 LM317, U10 SP-2U1+, U11 SMA, U12 LT1009, U13 TL974, U14 PMA4-33GLN+, U2 Teensy3.2, U3 SMA, U4 ROS-2536C-119+, U5 PMA4-33GLN+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

Commit message: Update
Parts:
- added TP9: TEST, Q2Footprint:PINTST, symbol TEST
- U11: footprint Q2Footprint:SMA -> Q2Footprint:SMA_Vertical
Connections:
- net at U2.18 (DAC), U4.2 (V-TUNE): now also TP9.1
Changed lines of the file:
@@
 LIBS:valves
 LIBS:Q2Lib
+LIBS:5-1814832-1
 LIBS:Q2-cache
 EELAYER 25 0
@@
 $EndComp
 $Comp
-L GND #PWR01
+L GND #PWR4
 U 1 1 5A7B7FE3
 P 1450 7100
-F 0 "#PWR01" H 1450 6850 50  0001 C CNN
+F 0 "#PWR4" H 1450 6850 50  0001 C CNN
 F 1 "GND" H 1450 6950 50  0000 C CNN
 F 2 "" H 1450 7100 50  0001 C CNN
@@
 $EndComp
 $Comp
-L GND #PWR02
+L GND #PWR1
 U 1 1 5A7B83F0
 P 800 1750
-F 0 "#PWR02" H 800 1500 50  0001 C CNN
+F 0 "#PWR1" H 800 1500 50  0001 C CNN
 F 1 "GND" H 800 1600 50  0000 C CNN
 F 2 "" H 800 1750 50  0001 C CNN
@@
 $EndComp
 $Comp
-L GND #PWR03
+L GND #PWR3
 U 1 1 5A7B870F
 P 1150 1800
-F 0 "#PWR03" H 1150 1550 50  0001 C CNN
+F 0 "#PWR3" H 1150 1550 50  0001 C CNN
 F 1 "GND" H 1150 1650 50  0000 C CNN
 F 2 "" H 1150 1800 50  0001 C CNN
@@
 $EndComp
 $Comp
-L GND #PWR04
+L GND #PWR5
 U 1 1 5A7B896E
 P 2600 1700
-F 0 "#PWR04" H 2600 1450 50  0001 C CNN
+F 0 "#PWR5" H 2600 1450 50  0001 C CNN
 F 1 "GND" H 2600 1550 50  0000 C CNN
 F 2 "" H 2600 1700 50  0001 C CNN
@@
 $EndComp
 $Comp
-L GND #PWR05
+L GND #PWR26
 U 1 1 5A7B8C7C
 P 10800 1350
-F 0 "#PWR05" H 10800 1100 50  0001 C CNN
+F 0 "#PWR26" H 10800 1100 50  0001 C CNN
 F 1 "GND" H 10800 1200 50  0000 C CNN
 F 2 "" H 10800 1350 50  0001 C CNN
@@
 NoConn ~ 11000 4050
 $Comp
-L GND #PWR06
+L GND #PWR27
 U 1 1 5A7BAB67
 P 12100 4150
-F 0 "#PWR06" H 12100 3900 50  0001 C CNN
+F 0 "#PWR27" H 12100 3900 50  0001 C CNN
 F 1 "GND" H 12100 4000 50  0000 C CNN
 F 2 "" H 12100 4150 50  0001 C CNN
@@
 +2.5V
 $Comp
-L GND #PWR07
+L GND #PWR7
 U 1 1 5A7D2EDC
 P 3350 8700
-F 0 "#PWR07" H 3350 8450 50  0001 C CNN
+F 0 "#PWR7" H 3350 8450 50  0001 C CNN
 F 1 "GND" H 3350 8550 50  0000 C CNN
 F 2 "" H 3350 8700 50  0001 C CNN
@@
 VCO
 $Comp
-L GND #PWR08
+L GND #PWR16
 U 1 1 5A7DA982
 P 5350 8750
-F 0 "#PWR08" H 5350 8500 50  0001 C CNN
+F 0 "#PWR16" H 5350 8500 50  0001 C CNN
 F 1 "GND" H 5350 8600 50  0000 C CNN
 F 2 "" H 5350 8750 50  0001 C CNN
@@
 $EndComp
 $Comp
-L GND #PWR09
+L GND #PWR22
 U 1 1 5A7C0AF4
 P 8300 8850
-F 0 "#PWR09" H 8300 8600 50  0001 C CNN
+F 0 "#PWR22" H 8300 8600 50  0001 C CNN
 F 1 "GND" H 8300 8700 50  0000 C CNN
 F 2 "" H 8300 8850 50  0001 C CNN
@@
 F 0 "U11" H 10400 8550 60  0000 C CNN
 F 1 "SMA" H 10400 8950 60  0000 C CNN
-F 2 "Q2Footprint:SMA" H 10450 8800 60  0001 C CNN
+F 2 "Q2Footprint:SMA_Vertical" H 10450 8800 60  0001 C CNN
 F 3 "" H 10450 8800 60  0001 C CNN
 	1    10400 8750
@@
 $EndComp
 $Comp
-L GND #PWR010
+L GND #PWR25
 U 1 1 5A7C6E17
 P 9950 8950
-F 0 "#PWR010" H 9950 8700 50  0001 C CNN
+F 0 "#PWR25" H 9950 8700 50  0001 C CNN
 F 1 "GND" H 9950 8800 50  0000 C CNN
 F 2 "" H 9950 8950 50  0001 C CNN
@@
 $EndComp
 $Comp
-L GND #PWR011
+L GND #PWR15
 U 1 1 5A7CCBCC
 P 4950 5600
-F 0 "#PWR011" H 4950 5350 50  0001 C CNN
+F 0 "#PWR15" H 4950 5350 50  0001 C CNN
 F 1 "GND" H 4950 5450 50  0000 C CNN
 F 2 "" H 4950 5600 50  0001 C CNN
@@
 $EndComp
 $Comp
-L GND #PWR012
+L GND #PWR13
 U 1 1 5A7CE644
 P 4750 5650
-F 0 "#PWR012" H 4750 5400 50  0001 C CNN
+F 0 "#PWR13" H 4750 5400 50  0001 C CNN
 F 1 "GND" H 4750 5500 50  0000 C CNN
 F 2 "" H 4750 5650 50  0001 C CNN
@@
 $EndComp
 $Comp
-L GND #PWR013
+L GND #PWR11
 U 1 1 5A7D1094
 P 4050 5750
-F 0 "#PWR013" H 4050 5500 50  0001 C CNN
+F 0 "#PWR11" H 4050 5500 50  0001 C CNN
 F 1 "GND" H 4050 5600 50  0000 C CNN
 F 2 "" H 4050 5750 50  0001 C CNN
@@
 $EndComp
 $Comp
-L GND #PWR014
+L GND #PWR6
 U 1 1 5A7D4CF2
 P 2900 5750
-F 0 "#PWR014" H 2900 5500 50  0001 C CNN
+F 0 "#PWR6" H 2900 5500 50  0001 C CNN
 F 1 "GND" H 2900 5600 50  0000 C CNN
 F 2 "" H 2900 5750 50  0001 C CNN
@@
 $EndComp
 $Comp
-L GND #PWR015
+L GND #PWR2
 U 1 1 5A7E1897
 P 1050 2850
-F 0 "#PWR015" H 1050 2600 50  0001 C CNN
+F 0 "#PWR2" H 1050 2600 50  0001 C CNN
 F 1 "GND" H 1050 2700 50  0000 C CNN
 F 2 "" H 1050 2850 50  0001 C CNN
@@
 $EndComp
 $Comp
-L GND #PWR016
+L GND #PWR9
 U 1 1 5A7E58BF
 P 3800 6250
-F 0 "#PWR016" H 3800 6000 50  0001 C CNN
+F 0 "#PWR9" H 3800 6000 50  0001 C CNN
 F 1 "GND" H 3800 6100 50  0000 C CNN
 F 2 "" H 3800 6250 50  0001 C CNN
@@
 $EndComp
 $Comp
-L GND #PWR017
+L GND #PWR21
 U 1 1 5A7F112C
 P 7100 6250
-F 0 "#PWR017" H 7100 6000 50  0001 C CNN
+F 0 "#PWR21" H 7100 6000 50  0001 C CNN
 F 1 "GND" H 7100 6100 50  0000 C CNN
 F 2 "" H 7100 6250 50  0001 C CNN
@@
 $EndComp
 $Comp
-L GND #PWR018
+L GND #PWR18
 U 1 1 5A80342D
 P 6750 6250
-F 0 "#PWR018" H 6750 6000 50  0001 C CNN
+F 0 "#PWR18" H 6750 6000 50  0001 C CNN
 F 1 "GND" H 6750 6100 50  0000 C CNN
 F 2 "" H 6750 6250 50  0001 C CNN
@@
 $EndComp
 $Comp
-L GND #PWR019
+L GND #PWR24
 U 1 1 5A806D56
 P 9550 7800
-F 0 "#PWR019" H 9550 7550 50  0001 C CNN
+F 0 "#PWR24" H 9550 7550 50  0001 C CNN
 F 1 "GND" H 9550 7650 50  0000 C CNN
 F 2 "" H 9550 7800 50  0001 C CNN
@@
 $EndComp
 $Comp
-L GND #PWR020
+L GND #PWR23
 U 1 1 5A80C661
 P 8350 3850
-F 0 "#PWR020" H 8350 3600 50  0001 C CNN
+F 0 "#PWR23" H 8350 3600 50  0001 C CNN
 F 1 "GND" H 8350 3700 50  0000 C CNN
 F 2 "" H 8350 3850 50  0001 C CNN
@@
 $EndComp
 $Comp
-L GND #PWR021
+L GND #PWR14
 U 1 1 5A7D8235
 P 4950 3800
-F 0 "#PWR021" H 4950 3550 50  0001 C CNN
+F 0 "#PWR14" H 4950 3550 50  0001 C CNN
 F 1 "GND" H 4950 3650 50  0000 C CNN
 F 2 "" H 4950 3800 50  0001 C CNN
@@
 $EndComp
 $Comp
-L GND #PWR022
+L GND #PWR12
 U 1 1 5A7D8241
 P 4750 3850
-F 0 "#PWR022" H 4750 3600 50  0001 C CNN
+F 0 "#PWR12" H 4750 3600 50  0001 C CNN
 F 1 "GND" H 4750 3700 50  0000 C CNN
 F 2 "" H 4750 3850 50  0001 C CNN
@@
 $EndComp
 $Comp
-L GND #PWR023
+L GND #PWR10
 U 1 1 5A7D8253
 P 4050 3950
-F 0 "#PWR023" H 4050 3700 50  0001 C CNN
+F 0 "#PWR10" H 4050 3700 50  0001 C CNN
 F 1 "GND" H 4050 3800 50  0000 C CNN
 F 2 "" H 4050 3950 50  0001 C CNN
@@
 $EndComp
 $Comp
-L GND #PWR024
+L GND #PWR8
 U 1 1 5A7D826B
 P 3800 4450
-F 0 "#PWR024" H 3800 4200 50  0001 C CNN
+F 0 "#PWR8" H 3800 4200 50  0001 C CNN
 F 1 "GND" H 3800 4300 50  0000 C CNN
 F 2 "" H 3800 4450 50  0001 C CNN
@@
 $EndComp
 $Comp
-L GND #PWR025
+L GND #PWR20
 U 1 1 5A7D8277
 P 7100 4450
-F 0 "#PWR025" H 7100 4200 50  0001 C CNN
+F 0 "#PWR20" H 7100 4200 50  0001 C CNN
 F 1 "GND" H 7100 4300 50  0000 C CNN
 F 2 "" H 7100 4450 50  0001 C CNN
@@
 $EndComp
 $Comp
-L GND #PWR026
+L GND #PWR17
 U 1 1 5A7D829C
 P 6750 4450
-F 0 "#PWR026" H 6750 4200 50  0001 C CNN
+F 0 "#PWR17" H 6750 4200 50  0001 C CNN
 F 1 "GND" H 6750 4300 50  0000 C CNN
 F 2 "" H 6750 4450 50  0001 C CNN
@@
 	12450 3450 12950 3450
 $Comp
-L GND #PWR027
+L GND #PWR19
 U 1 1 5A7E37D1
 P 6900 8900
-F 0 "#PWR027" H 6900 8650 50  0001 C CNN
+F 0 "#PWR19" H 6900 8650 50  0001 C CNN
 F 1 "GND" H 6900 8750 50  0000 C CNN
 F 2 "" H 6900 8900 50  0001 C CNN
@@
 Connection ~ 3150 7150
 Connection ~ 10100 3650
+$Comp
+L TEST TP9
+U 1 1 5A80FFAB
+P 3000 8550
+F 0 "TP9" H 3000 8850 50  0000 C BNN
+F 1 "TEST" H 3000 8800 50  0000 C CNN
+F 2 "Q2Footprint:PINTST" H 3000 8550 50  0001 C CNN
+F 3 "" H 3000 8550 50  0001 C CNN
+	1    3000 8550
+	1    0    0    -1
+$EndComp
+Connection ~ 3000 8550
 $EndSCHEMATC
